Commit message: tf树正常版本

File: src/four_wheel_robot_description/urdf/robot.urdf.xacro (robot description, xacro)
@@ -1,14 +1,15 @@
 <?xml version="1.0"?>
 <robot xmlns:xacro="http://www.ros.org/wiki/xacro" name="four_wheel_robot">
-    <!-- 包含机器人核心定义和传感器定义 -->
+    <!-- 包含文件 -->
     <xacro:include filename="$(find four_wheel_robot_description)/urdf/robot_core.xacro"/>
     <xacro:include filename="$(find four_wheel_robot_description)/urdf/sensors.xacro"/>
-    <!-- 添加3d激光雷达 -->
-    <xacro:lidar_3d_sensor name="velodyne"
-                          parent="base_link"
-                          xyz="0.2 0 ${chassis_height/2 + 0.05}"
-                          rpy="0 0 0"/>
+    <!-- 添加3D激光雷达 -->
+    <xacro:lidar_3d_sensor
+        name="laser_link"
+        parent="base_link"
+        xyz="0.2 0 ${chassis_height}"
+        rpy="0 0 0"/>
     <!-- 添加摄像头 -->
-   <xacro:stereo_camera_sensor name="stereo_camera"
+    <xacro:stereo_camera_sensor name="stereo_camera"
                                parent="base_link"
                                xyz="${chassis_length/2} 0 ${chassis_height/2}"
@@ -17,41 +18,3 @@
     <!-- 添加IMU -->
     <xacro:imu_sensor name="imu" parent="base_link" xyz="0 0 ${chassis_height/2}" rpy="0 0 0"/>
-    <!-- Gazebo颜色材质 -->
-    <gazebo reference="base_link">
-        <material>Gazebo/Blue</material>
-    </gazebo>
-    <gazebo reference="front_left_wheel">
-        <material>Gazebo/Black</material>
-    </gazebo>
-    <gazebo reference="front_right_wheel">
-        <material>Gazebo/Black</material>
-    </gazebo>
-    <gazebo reference="rear_left_wheel">
-        <material>Gazebo/Black</material>
-    </gazebo>
-    <gazebo reference="rear_right_wheel">
-        <material>Gazebo/Black</material>
-    </gazebo>
-    <!-- 差速驱动插件 -->
-    <gazebo>
-        <plugin name="diff_drive" filename="libgazebo_ros_diff_drive.so">
-            <left_joint>front_left_wheel_joint rear_left_wheel_joint</left_joint>
-            <right_joint>front_right_wheel_joint rear_right_wheel_joint</right_joint>
-            <wheel_separation>${chassis_width + wheel_width}</wheel_separation>
-            <wheel_diameter>${2 * wheel_radius}</wheel_diameter>
-            <max_wheel_torque>20</max_wheel_torque>
-            <max_wheel_acceleration>1.0</max_wheel_acceleration>
-            <odometry_frame>odom</odometry_frame>
-            <robot_base_frame>base_footprint</robot_base_frame>
-            <publish_odom>true</publish_odom>
-            <publish_odom_tf>true</publish_odom_tf>
-            <publish_wheel_tf>false</publish_wheel_tf>
-            <odometry_source>world</odometry_source>
-            <update_rate>30</update_rate>
-            <ros>
-                <remapping>cmd_vel:=cmd_vel</remapping>
-                <remapping>odom:=odom</remapping>
-            </ros>
-        </plugin>
-    </gazebo>
 </robot>

File: src/four_wheel_robot_description/urdf/robot_core.xacro (robot description, xacro)
@@ -7,4 +7,5 @@
     <xacro:property name="wheel_radius" value="0.1"/>
     <xacro:property name="wheel_width" value="0.05"/>
+    <xacro:property name="wheel_pos_x" value="0.25"/>  <!-- 前后轮距离车体中心的距离 -->
     <!-- 材质定义 -->
     <material name="blue">
@@ -14,34 +15,34 @@
         <color rgba="0 0 0 1"/>
     </material>
-    <!-- 添加底盘碰撞属性-->
-    <gazebo reference="base_link">
-        <material>Gazebo/Blue</material>
-        <mu1>0.2</mu1>
-        <mu2>0.2</mu2>
-        <selfCollide>true</selfCollide>
-        <gravity>true</gravity>
-        <!-- 添加碰撞传感器 -->
-        <sensor name="contact_sensor" type="contact">
-            <always_on>true</always_on>
-            <update_rate>30.0</update_rate>
-            <contact>
-                <collision>base_link_collision</collision>
-            </contact>
-            <plugin name="gazebo_ros_bumper_controller" filename="libgazebo_ros_bumper.so">
-                <ros>
-                    <remapping>~/bumper_states:=bumper_states</remapping>
-                </ros>
-                <frame_name>base_link</frame_name>
-            </plugin>
-        </sensor>
-    </gazebo>
-    <!-- 添加基座链接 -->
-    <link name="base_footprint"/>
-    <joint name="base_joint" type="fixed">
-        <parent link="base_footprint"/>
-        <child link="base_link"/>
-        <origin xyz="0 0 ${wheel_radius}" rpy="0 0 0"/>
+    <!-- Base Footprint -->
+    <link name="base_footprint">
+        <inertial>
+            <mass value="0.0001"/>
+            <origin xyz="0 0 0" rpy="0 0 0"/>
+            <inertia
+                ixx="0.0001" ixy="0.0" ixz="0.0"
+                iyy="0.0001" iyz="0.0"
+                izz="0.0001"/>
+        </inertial>
+        <visual>
+            <origin xyz="0 0 0" rpy="0 0 0"/>
+            <geometry>
+                <box size="0.001 0.001 0.001"/>
+            </geometry>
+        </visual>
+        <collision>
+            <origin xyz="0 0 0" rpy="0 0 0"/>
+            <geometry>
+                <box size="0.001 0.001 0.001"/>
+            </geometry>
+        </collision>
+    </link>
+    <!-- base_link 到 base_footprint 的固定关节 -->
+    <joint name="base_link_to_footprint" type="fixed">
+        <parent link="base_link"/>
+        <child link="base_footprint"/>
+        <origin xyz="0 0 -${wheel_radius}" rpy="0 0 0"/>
     </joint>
-    <!-- 底盘link -->
+    <!-- 底盘 Base Link -->
     <link name="base_link">
         <visual>
@@ -59,14 +60,19 @@
         </collision>
         <inertial>
-            <mass value="1.0"/>
+            <mass value="5.0"/>
             <origin xyz="0 0 ${chassis_height/2}" rpy="0 0 0"/>
-            <inertia ixx="0.1" ixy="0" ixz="0"
-                     iyy="0.1" iyz="0"
-                     izz="0.1"/>
+            <inertia
+                ixx="${(1/12) * 5.0 * (chassis_width*chassis_width + chassis_height*chassis_height)}"
+                ixy="0"
+                ixz="0"
+                iyy="${(1/12) * 5.0 * (chassis_length*chassis_length + chassis_height*chassis_height)}"
+                iyz="0"
+                izz="${(1/12) * 5.0 * (chassis_length*chassis_length + chassis_width*chassis_width)}"/>
         </inertial>
     </link>
-    <!-- 更新车轮碰撞属性 -->
+    <!-- 车轮宏定义 -->
     <xacro:macro name="wheel" params="prefix x_offset y_offset">
-      <link name="${prefix}_wheel">
+        <!-- 轮子link -->
+        <link name="${prefix}_wheel">
             <visual>
                 <geometry>
@@ -74,4 +80,5 @@
                 </geometry>
                 <material name="black"/>
+                <origin xyz="0 0 0" rpy="${pi/2} 0 0"/>
             </visual>
             <collision>
@@ -79,8 +86,16 @@
                     <cylinder radius="${wheel_radius}" length="${wheel_width}"/>
                 </geometry>
+                <origin xyz="0 0 0" rpy="${pi/2} 0 0"/>
             </collision>
             <inertial>
                 <mass value="0.5"/>
-                <inertia ixx="0.01" ixy="0" ixz="0" iyy="0.01" iyz="0" izz="0.01"/>
+                <origin xyz="0 0 0" rpy="${pi/2} 0 0"/>
+                <inertia
+                    ixx="${(1/12) * 0.5 * (3*wheel_radius*wheel_radius + wheel_width*wheel_width)}"
+                    ixy="0"
+                    ixz="0"
+                    iyy="${(1/12) * 0.5 * (3*wheel_radius*wheel_radius + wheel_width*wheel_width)}"
+                    iyz="0"
+                    izz="${(1/2) * 0.5 * (wheel_radius*wheel_radius)}"/>
             </inertial>
         </link>
@@ -88,22 +103,62 @@
             <parent link="base_link"/>
             <child link="${prefix}_wheel"/>
-            <origin xyz="${x_offset} ${y_offset} 0" rpy="${pi/2} 0 0"/>
-            <axis xyz="0 0 1"/>
+            <origin xyz="${x_offset} ${y_offset} 0" rpy="0 0 0"/>
+            <axis xyz="0 1 0"/>
         </joint>
+        <!-- Gazebo specific wheel properties -->
         <gazebo reference="${prefix}_wheel">
             <material>Gazebo/Black</material>
-            <mu1>1.0</mu1>
-            <mu2>1.0</mu2>
-            <kp>1000000.0</kp>
-            <kd>100.0</kd>
+            <mu1>0.8</mu1>
+            <mu2>0.8</mu2>
+            <kp>500000.0</kp>
+            <kd>50.0</kd>
             <minDepth>0.001</minDepth>
-            <maxVel>1.0</maxVel>
+            <maxVel>1.5</maxVel>
             <fdir1>1 0 0</fdir1>
         </gazebo>
+        <!-- 添加传动装置 -->
+        <transmission name="${prefix}_wheel_trans">
+            <type>transmission_interface/SimpleTransmission</type>
+            <joint name="${prefix}_wheel_joint">
+                <hardwareInterface>hardware_interface/VelocityJointInterface</hardwareInterface>
+            </joint>
+            <actuator name="${prefix}_wheel_motor">
+                <mechanicalReduction>1</mechanicalReduction>
+            </actuator>
+        </transmission>
     </xacro:macro>
-    <!-- 使用宏创建四个轮子 -->
-    <xacro:wheel prefix="front_left" x_offset="${chassis_length/4}" y_offset="${chassis_width/2 + wheel_width/2}"/>
-    <xacro:wheel prefix="front_right" x_offset="${chassis_length/4}" y_offset="-${chassis_width/2 + wheel_width/2}"/>
-    <xacro:wheel prefix="rear_left" x_offset="-${chassis_length/4}" y_offset="${chassis_width/2 + wheel_width/2}"/>
-    <xacro:wheel prefix="rear_right" x_offset="-${chassis_length/4}" y_offset="-${chassis_width/2 + wheel_width/2}"/>
+    <!-- 使用wheel_pos_x参数统一轮子位置 -->
+    <xacro:wheel prefix="front_left" x_offset="${wheel_pos_x}" y_offset="${chassis_width/2 + wheel_width/2}"/>
+    <xacro:wheel prefix="front_right" x_offset="${wheel_pos_x}" y_offset="-${chassis_width/2 + wheel_width/2}"/>
+    <xacro:wheel prefix="rear_left" x_offset="-${wheel_pos_x}" y_offset="${chassis_width/2 + wheel_width/2}"/>
+    <xacro:wheel prefix="rear_right" x_offset="-${wheel_pos_x}" y_offset="-${chassis_width/2 + wheel_width/2}"/>
+    <gazebo reference="base_link">
+        <material>Gazebo/Blue</material>
+        <mu1>0.2</mu1>
+        <mu2>0.2</mu2>
+        <kp>1000000.0</kp>
+        <kd>100.0</kd>
+    </gazebo>
+    <!-- 差速驱动插件配置 -->
+    <gazebo>
+        <plugin name="diff_drive" filename="libgazebo_ros_diff_drive.so">
+            <!-- 基本配置 -->
+            <ros>
+                <namespace>/</namespace>
+                <remapping>cmd_vel:=cmd_vel</remapping>
+                <remapping>odom:=odom</remapping>
+            </ros>
+            <!-- 轮子配置 -->
+            <left_joint>front_left_wheel_joint</left_joint>
+            <right_joint>front_right_wheel_joint</right_joint>
+            <wheel_separation>0.4</wheel_separation>
+            <wheel_diameter>0.2</wheel_diameter>
+            <!-- 发布TF和里程计 -->
+            <publish_odom>true</publish_odom>
+            <publish_odom_tf>true</publish_odom_tf>
+            <publish_wheel_tf>true</publish_wheel_tf>
+            <odometry_frame>odom</odometry_frame>
+            <robot_base_frame>base_link</robot_base_frame>
+        </plugin>
+    </gazebo>
 </robot>

File: src/four_wheel_robot_description/urdf/sensors.xacro (robot description, xacro)
@@ -3,10 +3,12 @@
     <!-- 3D LiDAR宏定义 -->
     <xacro:macro name="lidar_3d_sensor" params="name parent xyz rpy">
+        <!-- 激光雷达关节 -->
         <joint name="${name}_joint" type="fixed">
             <parent link="${parent}"/>
-            <child link="${name}_link"/>
+            <child link="${name}"/>
             <origin xyz="${xyz}" rpy="${rpy}"/>
         </joint>
-        <link name="${name}_link">
+        <!-- 激光雷达连杆 -->
+        <link name="${name}">
             <visual>
                 <geometry>
@@ -21,17 +23,24 @@
             </collision>
             <inertial>
-                <mass value="0.8"/>
-                <inertia ixx="0.001" ixy="0" ixz="0" iyy="0.001" iyz="0" izz="0.001"/>
+                <mass value="0.1"/>
+                <origin xyz="0 0 0" rpy="0 0 0"/>
+                <inertia
+                    ixx="0.001"
+                    ixy="0"
+                    ixz="0"
+                    iyy="0.001"
+                    iyz="0"
+                    izz="0.001"/>
             </inertial>
         </link>
-        <gazebo reference="${name}_link">
+        <gazebo reference="${name}">
             <sensor type="ray" name="${name}">
-                <pose>0 0 0 0 0 0</pose>
-                <visualize>false</visualize>
+                <always_on>true</always_on>
+                <visualize>true</visualize>
                 <update_rate>10</update_rate>
                 <ray>
                     <scan>
                         <horizontal>
-                            <samples>1800</samples>
+                            <samples>360</samples>
                             <resolution>1</resolution>
                             <min_angle>-3.14159</min_angle>
@@ -47,5 +56,5 @@
                     <range>
                         <min>0.3</min>
-                        <max>100.0</max>
+                        <max>30.0</max>
                         <resolution>0.01</resolution>
                     </range>
@@ -53,15 +62,16 @@
                 <plugin name="${name}_controller" filename="libgazebo_ros_ray_sensor.so">
                     <ros>
-                        <namespace>/${name}</namespace>
-                        <remapping>~/out:=points</remapping>
+                        <namespace>/four_wheel_robot</namespace>
+                        <remapping>~/out:=scan</remapping>
                     </ros>
                     <output_type>sensor_msgs/PointCloud2</output_type>
-                    <frame_name>${name}_link</frame_name>
+                    <frame_name>${name}</frame_name>
                 </plugin>
             </sensor>
         </gazebo>
     </xacro:macro>
-    <!-- 立体相机宏定义 -->
+    <!-- Stereo Camera 宏定义 -->
     <xacro:macro name="stereo_camera_sensor" params="name parent xyz rpy baseline">
+        <!-- 相机基座链接 -->
         <joint name="${name}_joint" type="fixed">
             <parent link="${parent}"/>
@@ -72,20 +82,48 @@
             <visual>
                 <geometry>
-                    <box size="0.02 ${baseline + 0.02} 0.02"/>
-                </geometry>
-                <material name="red"/>
+                    <box size="0.02 0.02 0.02"/>
+                </geometry>
+                <material name="black"/>
             </visual>
             <collision>
                 <geometry>
-                    <box size="0.02 ${baseline + 0.02} 0.02"/>
+                    <box size="0.02 0.02 0.02"/>
                 </geometry>
             </collision>
             <inertial>
-                <mass value="0.2"/>
+                <mass value="0.1"/>
                 <inertia ixx="0.001" ixy="0" ixz="0" iyy="0.001" iyz="0" izz="0.001"/>
             </inertial>
         </link>
         <!-- 左相机 -->
-        <gazebo reference="${name}_link">
+        <joint name="${name}_left_joint" type="fixed">
+            <parent link="${name}_link"/>
+            <child link="${name}_left"/>
+            <origin xyz="0 ${baseline/2} 0" rpy="0 0 0"/>
+        </joint>
+        <link name="${name}_left">
+            <visual>
+                <geometry>
+                    <box size="0.01 0.01 0.01"/>
+                </geometry>
+                <material name="black"/>
+            </visual>
+        </link>
+        <!-- 右相机 -->
+        <joint name="${name}_right_joint" type="fixed">
+            <parent link="${name}_link"/>
+            <child link="${name}_right"/>
+            <origin xyz="0 -${baseline/2} 0" rpy="0 0 0"/>
+        </joint>
+        <link name="${name}_right">
+            <visual>
+                <geometry>
+                    <box size="0.01 0.01 0.01"/>
+                </geometry>
+                <material name="black"/>
+            </visual>
+        </link>
+        <!-- Gazebo插件配置 -->
+        <gazebo reference="${name}_left">
             <sensor type="camera" name="${name}_left">
                 <update_rate>30.0</update_rate>
@@ -98,27 +136,18 @@
                     </image>
                     <clip>
-                        <near>0.02</near>
-                        <far>300</far>
+                        <near>0.1</near>
+                        <far>100.0</far>
                     </clip>
-                    <noise>
-                        <type>gaussian</type>
-                        <mean>0.0</mean>
-                        <stddev>0.007</stddev>
-                    </noise>
                 </camera>
                 <plugin name="${name}_left_controller" filename="libgazebo_ros_camera.so">
                     <ros>
-                        <namespace>/${name}</namespace>
-                        <remapping>image_raw:=left/image_raw</remapping>
-                        <remapping>camera_info:=left/camera_info</remapping>
-                    </ros>
-                    <camera_name>left</camera_name>
-                    <frame_name>${name}_link</frame_name>
-                    <hack_baseline>0.0</hack_baseline>
-                </plugin>
-            </sensor>
-        </gazebo>
-        <!-- 右相机 -->
-        <gazebo reference="${name}_link">
+                        <namespace>/four_wheel_robot</namespace>
+                        <remapping>image_raw:=${name}_left/image_raw</remapping>
+                    </ros>
+                    <frame_name>${name}_left</frame_name>
+                </plugin>
+            </sensor>
+        </gazebo>
+        <gazebo reference="${name}_right">
             <sensor type="camera" name="${name}_right">
                 <update_rate>30.0</update_rate>
@@ -131,61 +160,47 @@
                     </image>
                     <clip>
-                        <near>0.02</near>
-                        <far>300</far>
+                        <near>0.1</near>
+                        <far>100.0</far>
                     </clip>
-                    <noise>
-                        <type>gaussian</type>
-                        <mean>0.0</mean>
-                        <stddev>0.007</stddev>
-                    </noise>
                 </camera>
                 <plugin name="${name}_right_controller" filename="libgazebo_ros_camera.so">
                     <ros>
-                        <namespace>/${name}</namespace>
-                        <remapping>image_raw:=right/image_raw</remapping>
-                        <remapping>camera_info:=right/camera_info</remapping>
-                    </ros>
-                    <camera_name>right</camera_name>
-                    <frame_name>${name}_link</frame_name>
-                    <hack_baseline>${baseline}</hack_baseline>
+                        <namespace>/four_wheel_robot</namespace>
+                        <remapping>image_raw:=${name}_right/image_raw</remapping>
+                    </ros>
+                    <frame_name>${name}_right</frame_name>
                 </plugin>
             </sensor>
         </gazebo>
     </xacro:macro>
-    <!-- IMU宏定义 -->
+    <!-- IMU 宏定义 -->
     <xacro:macro name="imu_sensor" params="name parent xyz rpy">
         <joint name="${name}_joint" type="fixed">
             <parent link="${parent}"/>
-            <child link="${name}_link"/>
+            <child link="${name}"/>
             <origin xyz="${xyz}" rpy="${rpy}"/>
         </joint>
-        <link name="${name}_link">
-            <visual>
-                <geometry>
-                    <box size="0.02 0.02 0.02"/>
-                </geometry>
-                <material name="red"/>
-            </visual>
-            <collision>
-                <geometry>
-                    <box size="0.02 0.02 0.02"/>
-                </geometry>
-            </collision>
+        <link name="${name}">
             <inertial>
-                <mass value="0.1"/>
-                <inertia ixx="0.001" ixy="0" ixz="0" iyy="0.001" iyz="0" izz="0.001"/>
+                <mass value="0.001"/>
+                <origin xyz="0 0 0" rpy="0 0 0"/>
+                <inertia ixx="0.0001" ixy="0" ixz="0" iyy="0.0001" iyz="0" izz="0.0001"/>
             </inertial>
         </link>
-        <gazebo reference="${name}_link">
-            <sensor type="imu" name="${name}">
+        <gazebo reference="${name}">
+            <sensor name="${name}_sensor" type="imu">
                 <always_on>true</always_on>
                 <update_rate>100</update_rate>
                 <visualize>true</visualize>
-                <plugin name="${name}_controller" filename="libgazebo_ros_imu_sensor.so">
-                    <ros>
-                        <namespace>/${name}</namespace>
-                        <remapping>~/out:=data</remapping>
-                    </ros>
-                    <frame_name>${name}_link</frame_name>
+                <plugin name="imu_plugin" filename="libgazebo_ros_imu_sensor.so">
+                    <ros>
+                        <namespace>/</namespace>
+                        <remapping>~/out:=imu</remapping>
+                    </ros>
+                    <initial_orientation_as_reference>false</initial_orientation_as_reference>
+                    <frame_name>${name}</frame_name>
+                    <xyzOffset>0 0 0</xyzOffset>
+                    <rpyOffset>0 0 0</rpyOffset>
+                    <gaussianNoise>0.00001</gaussianNoise>
                 </plugin>
             </sensor>
